Commit message: current_limit

File: src/arm/robot_arm_description/urdf/manual_total_robot.urdf.xacro (robot description, xacro)
@@ -140,5 +140,5 @@
     <origin xyz="0 0 0.182" rpy="0 0 0"/>
   </joint>
-  <xacro:macro name="rmd_actuator" params="name joint_name actuator_id max_velocity">
+  <xacro:macro name="rmd_actuator" params="name joint_name actuator_id max_velocity current_limit current_release">
     <ros2_control name="${name}" type="actuator">
       <hardware>
@@ -147,4 +147,9 @@
         <param name="torque_constant">1.0</param><param name="max_velocity">${max_velocity}</param>
         <param name="velocity_alpha">0.1</param><param name="effort_alpha">0.1</param>
+        <param name="software_current_limit">${current_limit}</param>
+        <param name="current_release_threshold">${current_release}</param>
+        <param name="current_limit_duration_ms">50</param>
+        <param name="current_retreat_velocity">0.1</param>
+        <param name="current_max_retreat_distance">0.174533</param>
         <param name="timeout">$(arg timeout)</param>
       </hardware>
@@ -155,7 +160,7 @@
     </ros2_control>
   </xacro:macro>
-  <xacro:rmd_actuator name="shoulder_rmd" joint_name="shoulder_lift_joint" actuator_id="$(arg shoulder_actuator_id)" max_velocity="$(arg shoulder_max_velocity)"/>
-  <xacro:rmd_actuator name="elbow_rmd" joint_name="elbow_joint" actuator_id="$(arg elbow_actuator_id)" max_velocity="$(arg elbow_max_velocity)"/>
-  <xacro:rmd_actuator name="wrist_rmd" joint_name="wrist_joint" actuator_id="$(arg wrist_actuator_id)" max_velocity="$(arg wrist_max_velocity)"/>
+  <xacro:rmd_actuator name="shoulder_rmd" joint_name="shoulder_lift_joint" actuator_id="$(arg shoulder_actuator_id)" max_velocity="$(arg shoulder_max_velocity)" current_limit="10.0" current_release="8.5"/>
+  <xacro:rmd_actuator name="elbow_rmd" joint_name="elbow_joint" actuator_id="$(arg elbow_actuator_id)" max_velocity="$(arg elbow_max_velocity)" current_limit="8.0" current_release="6.8"/>
+  <xacro:rmd_actuator name="wrist_rmd" joint_name="wrist_joint" actuator_id="$(arg wrist_actuator_id)" max_velocity="$(arg wrist_max_velocity)" current_limit="4.0" current_release="3.4"/>
   <ros2_control name="dynamixel_system" type="system">
     <hardware>

File: src/arm/robot_arm_description/urdf/test_urdf.urdf.xacro (robot description, xacro)
@@ -19,5 +19,5 @@
     </inertial>
   </xacro:macro>
-  <xacro:macro name="rmd_actuator" params="name joint_name actuator_id torque_constant">
+  <xacro:macro name="rmd_actuator" params="name joint_name actuator_id torque_constant current_limit current_release">
     <ros2_control name="${name}" type="actuator">
       <hardware>
@@ -29,4 +29,9 @@
         <param name="velocity_alpha">0.1</param>
         <param name="effort_alpha">0.1</param>
+        <param name="software_current_limit">${current_limit}</param>
+        <param name="current_release_threshold">${current_release}</param>
+        <param name="current_limit_duration_ms">50</param>
+        <param name="current_retreat_velocity">0.1</param>
+        <param name="current_max_retreat_distance">0.174533</param>
         <param name="timeout">$(arg timeout)</param>
       </hardware>
@@ -122,12 +127,15 @@
   <xacro:rmd_actuator name="shoulder_rmd" joint_name="shoulder_lift_joint"
                       actuator_id="$(arg shoulder_actuator_id)"
-                      torque_constant="$(arg shoulder_torque_constant)"/>
+                      torque_constant="$(arg shoulder_torque_constant)"
+                      current_limit="10.0" current_release="8.5"/>
   <xacro:rmd_actuator name="elbow_rmd" joint_name="elbow_joint"
                       actuator_id="$(arg elbow_actuator_id)"
-                      torque_constant="$(arg elbow_torque_constant)"/>
+                      torque_constant="$(arg elbow_torque_constant)"
+                      current_limit="8.0" current_release="6.8"/>
   <!-- wrist 하드웨어 세팅 전까지 CAN 액추에이터 등록을 비활성화합니다.
   <xacro:rmd_actuator name="wrist_rmd" joint_name="wrist_joint"
                       actuator_id="$(arg wrist_actuator_id)"
-                      torque_constant="$(arg wrist_torque_constant)"/>
+                      torque_constant="$(arg wrist_torque_constant)"
+                      current_limit="4.0" current_release="3.4"/>
   -->
 </robot>

Commit message: 다이나믹셀 수정2

File: src/arm/robot_arm_description/urdf/manual_total_robot.urdf.xacro (robot description, xacro)
@@ -48,5 +48,5 @@
     <parent link="base_link"/><child link="base_yaw_link"/>
     <origin xyz="0 0 ${sh_off}" rpy="0 0 0"/><axis xyz="0 0 1"/>
-    <limit lower="-3.1416" upper="3.1416" effort="3.1" velocity="2.618"/>
+    <limit lower="-1.5708" upper="1.5708" effort="3.1" velocity="2.618"/>
     <dynamics damping="0.05" friction="0.02"/>
   </joint>
